File: kicad/dev/px16_regfile/px16_regfile.kicad_pcb (KiCad board)
At the start: 2 copper layers, 195 parts, among them J1 Conn_02x12_Odd_Even, J2 Conn_02x12_Odd_Even, J3 Conn_02x12_Odd_Even, J4 Screw_Terminal_01x02, U1 74LS273, U10 74LS273, U11 74LS244, U12 74LS244, U13 74LS273, U14 74LS244, U15 74LS244, U16 74LS273, U17 74LS244, U18 74LS244, U19 74LS273, U2 74LS244, U20 74LS244, U21 74LS244, U22 74LS273, U23 74LS244, U24 74LS244, U25 74LS273, U26 74LS244, U27 74LS244, U28 74LS273, U29 74LS244, U3 74LS244, U30 74LS244, U4 74LS273, U5 74LS244, U6 74LS244, U7 74LS273, U8 74LS244, U9 74LS244

Commit message: Work on PC and PF in regfile.
Parts:
- added D100: LED, LED_THT:LED_D5.0mm, F.Cu at (748.3, 279.4)
- added D101: LED, LED_THT:LED_D5.0mm, F.Cu at (711.6, 301.3)
- added D102: LED, LED_THT:LED_D5.0mm, F.Cu at (726.6, 298.8)
- added D103: LED, LED_THT:LED_D5.0mm, F.Cu at (748.3, 271.9)
- added D81: LED, LED_THT:LED_D5.0mm, F.Cu at (715.7, 308.9)
- added D82: LED, LED_THT:LED_D5.0mm, F.Cu at (697.4, 328.3)
- added D83: LED, LED_THT:LED_D5.0mm, F.Cu at (740.8, 271.9)
- added D84: LED, LED_THT:LED_D5.0mm, F.Cu at (733.3, 271.9)
- added D85: LED, LED_THT:LED_D5.0mm, F.Cu at (689.9, 320.8)
- added D86: LED, LED_THT:LED_D5.0mm, F.Cu at (733.3, 279.4)
- added D87: LED, LED_THT:LED_D5.0mm, F.Cu at (726.6, 291.3)
- added D88: LED, LED_THT:LED_D5.0mm, F.Cu at (689.9, 328.3)
- added D89: LED, LED_THT:LED_D5.0mm, F.Cu at (740.8, 279.4)
- added D90: LED, LED_THT:LED_D5.0mm, F.Cu at (755.8, 271.9)
- added D91: LED, LED_THT:LED_D5.0mm, F.Cu at (708.2, 313.2)
- added D92: LED, LED_THT:LED_D5.0mm, F.Cu at (708.2, 320.7)
- added D93: LED, LED_THT:LED_D5.0mm, F.Cu at (689.9, 335.9)
- added D94: LED, LED_THT:LED_D5.0mm, F.Cu at (700.7, 313.2)
- added D95: LED, LED_THT:LED_D5.0mm, F.Cu at (719.1, 293.8)
- added D96: LED, LED_THT:LED_D5.0mm, F.Cu at (711.6, 293.8)
- added D97: LED, LED_THT:LED_D5.0mm, F.Cu at (700.7, 320.7)
- added D98: LED, LED_THT:LED_D5.0mm, F.Cu at (734.1, 287.0)
- added D99: LED, LED_THT:LED_D5.0mm, F.Cu at (719.1, 301.3)
- added J5: Conn_02x12_Odd_Even, Connector_PinHeader_2.54mm:PinHeader_2x12_P2.54mm_Vertical, F.Cu at (628.3, 303.0)
- added J6: Conn_02x12_Odd_Even, Connector_PinHeader_2.54mm:PinHeader_2x12_P2.54mm_Vertical, F.Cu at (628.3, 270.4)
- added R100: R, Resistor_THT:R_Axial_DIN0207_L6.3mm_D2.5mm_P2.54mm_Vertical, F.Cu at (733.6, 292.8)
- added R101: R, Resistor_THT:R_Axial_DIN0207_L6.3mm_D2.5mm_P2.54mm_Vertical, F.Cu at (704.4, 326.5)
- added R102: R, Resistor_THT:R_Axial_DIN0207_L6.3mm_D2.5mm_P2.54mm_Vertical, F.Cu at (628.0, 343.4)
- added R103: R, Resistor_THT:R_Axial_DIN0207_L6.3mm_D2.5mm_P2.54mm_Vertical, F.Cu at (722.8, 311.2)
- added R81: R, Resistor_THT:R_Axial_DIN0207_L6.3mm_D2.5mm_P2.54mm_Vertical, F.Cu at (678.6, 343.5)
- added R82: R, Resistor_THT:R_Axial_DIN0207_L6.3mm_D2.5mm_P2.54mm_Vertical, F.Cu at (690.9, 345.7)
- added R83: R, Resistor_THT:R_Axial_DIN0207_L6.3mm_D2.5mm_P2.54mm_Vertical, F.Cu at (755.3, 277.7)
- added R84: R, Resistor_THT:R_Axial_DIN0207_L6.3mm_D2.5mm_P2.54mm_Vertical, F.Cu at (704.4, 330.6)
- added R85: R, Resistor_THT:R_Axial_DIN0207_L6.3mm_D2.5mm_P2.54mm_Vertical, F.Cu at (628.0, 339.4)
- added R86: R, Resistor_THT:R_Axial_DIN0207_L6.3mm_D2.5mm_P2.54mm_Vertical, F.Cu at (628.0, 335.3)
- added R87: R, Resistor_THT:R_Axial_DIN0207_L6.3mm_D2.5mm_P2.54mm_Vertical, F.Cu at (722.8, 307.1)
- added R88: R, Resistor_THT:R_Axial_DIN0207_L6.3mm_D2.5mm_P2.54mm_Vertical, F.Cu at (762.8, 270.1)
- added R89: R, Resistor_THT:R_Axial_DIN0207_L6.3mm_D2.5mm_P2.54mm_Vertical, F.Cu at (739.8, 292.8)
- added R90: R, Resistor_THT:R_Axial_DIN0207_L6.3mm_D2.5mm_P2.54mm_Vertical, F.Cu at (715.3, 318.7)
- added R91: R, Resistor_THT:R_Axial_DIN0207_L6.3mm_D2.5mm_P2.54mm_Vertical, F.Cu at (733.6, 296.8)
- added R92: R, Resistor_THT:R_Axial_DIN0207_L6.3mm_D2.5mm_P2.54mm_Vertical, F.Cu at (741.1, 285.2)
- added R93: R, Resistor_THT:R_Axial_DIN0207_L6.3mm_D2.5mm_P2.54mm_Vertical, F.Cu at (747.3, 285.2)
- added R94: R, Resistor_THT:R_Axial_DIN0207_L6.3mm_D2.5mm_P2.54mm_Vertical, F.Cu at (733.6, 300.9)
- added R95: R, Resistor_THT:R_Axial_DIN0207_L6.3mm_D2.5mm_P2.54mm_Vertical, F.Cu at (684.7, 343.5)
- added R96: R, Resistor_THT:R_Axial_DIN0207_L6.3mm_D2.5mm_P2.54mm_Vertical, F.Cu at (715.3, 314.7)
- added R97: R, Resistor_THT:R_Axial_DIN0207_L6.3mm_D2.5mm_P2.54mm_Vertical, F.Cu at (696.9, 334.1)
- added R98: R, Resistor_THT:R_Axial_DIN0207_L6.3mm_D2.5mm_P2.54mm_Vertical, F.Cu at (690.9, 341.7)
- added R99: R, Resistor_THT:R_Axial_DIN0207_L6.3mm_D2.5mm_P2.54mm_Vertical, F.Cu at (710.6, 326.5)
- added U31: 74LS139, Package_DIP:DIP-16_W7.62mm, F.Cu at (710.7, 270.2)
- added U32: 74LS04, Package_DIP:DIP-14_W7.62mm, F.Cu at (699.9, 292.1)
- added U33: 74LS139, Package_DIP:DIP-16_W7.62mm, F.Cu at (645.6, 324.2)
- added U34: 74LS139, Package_DIP:DIP-16_W7.62mm, F.Cu at (699.9, 270.2)
- added U35: 74LS02, Package_DIP:DIP-14_W7.62mm, F.Cu at (721.6, 270.2)
- added U36: 74LS02, Package_DIP:DIP-14_W7.62mm, F.Cu at (678.2, 324.2)
- added U37: 74LS273, Package_DIP:DIP-20_W7.62mm, F.Cu at (645.6, 270.2)
- added U38: 74LS244, Package_DIP:DIP-20_W7.62mm, F.Cu at (667.3, 270.2)
- added U39: 74LS244, Package_DIP:DIP-20_W7.62mm, F.Cu at (634.8, 270.2)
- added U40: 74LS244, Package_DIP:DIP-20_W7.62mm, F.Cu at (678.2, 297.2)
- added U41: 74LS244, Package_DIP:DIP-20_W7.62mm, F.Cu at (678.2, 270.2)
- added U42: 74LS244, Package_DIP:DIP-20_W7.62mm, F.Cu at (645.6, 297.2)
- added U43: 74LS244, Package_DIP:DIP-20_W7.62mm, F.Cu at (656.5, 297.2)
- added U44: 74LS161, Package_DIP:DIP-16_W7.62mm, F.Cu at (634.8, 324.2)
- added U45: 74LS161, Package_DIP:DIP-16_W7.62mm, F.Cu at (689.0, 297.2)
- added U46: 74LS244, Package_DIP:DIP-20_W7.62mm, F.Cu at (667.3, 297.2)
- added U47: 74LS244, Package_DIP:DIP-20_W7.62mm, F.Cu at (656.5, 270.2)
- added U48: 74LS161, Package_DIP:DIP-16_W7.62mm, F.Cu at (667.3, 324.2)
- added U49: 74LS161, Package_DIP:DIP-16_W7.62mm, F.Cu at (656.5, 324.2)
- added U50: 74LS244, Package_DIP:DIP-20_W7.62mm, F.Cu at (689.0, 270.2)
- added U51: 74LS244, Package_DIP:DIP-20_W7.62mm, F.Cu at (634.8, 297.2)
Connections:
- U1 pad 1: unconnected-(U1-Pad1) -> /~{RST}
- U1 pad 11: unconnected-(U1-Pad11) -> /R0-WE
- U10 pad 1: unconnected-(U10-Pad1) -> /~{RST}
- U10 pad 11: unconnected-(U10-Pad11) -> /R1-WE
- U11 pad 1: Net-(U11-Pad1) -> /~{R1-OEa}
- U11 pad 19: Net-(U11-Pad1) -> /~{R1-OEa}
- U12 pad 1: Net-(U11-Pad1) -> /~{R1-OEb}
- U12 pad 19: Net-(U11-Pad1) -> /~{R1-OEb}
- U13 pad 1: unconnected-(U13-Pad1) -> /~{RST}
- U13 pad 11: unconnected-(U13-Pad11) -> /R2-WE
- U14 pad 1: Net-(U14-Pad1) -> /~{R2-OEa}
- U14 pad 19: Net-(U14-Pad1) -> /~{R2-OEa}
- U15 pad 1: Net-(U14-Pad1) -> /~{R2-OEb}
- U15 pad 19: Net-(U14-Pad1) -> /~{R2-OEb}
- U16 pad 1: unconnected-(U16-Pad1) -> /~{RST}
- U16 pad 11: unconnected-(U16-Pad11) -> /R2-WE
- U17 pad 1: Net-(U17-Pad1) -> /~{R2-OEa}
- U17 pad 19: Net-(U17-Pad1) -> /~{R2-OEa}
- U18 pad 1: Net-(U17-Pad1) -> /~{R2-OEb}
- U18 pad 19: Net-(U17-Pad1) -> /~{R2-OEb}
- U19 pad 1: unconnected-(U19-Pad1) -> /~{RST}
- U19 pad 11: unconnected-(U19-Pad11) -> /R3-WE
- U2 pad 1: Net-(U2-Pad1) -> /~{R0-OEa}
- U2 pad 19: Net-(U2-Pad1) -> /~{R0-OEa}
- U20 pad 1: Net-(U20-Pad1) -> /~{R3-OEa}
- U20 pad 19: Net-(U20-Pad1) -> /~{R3-OEa}
- U21 pad 1: Net-(U21-Pad1) -> /~{R3-OEb}
- U21 pad 19: Net-(U21-Pad1) -> /~{R3-OEb}
- U22 pad 1: unconnected-(U22-Pad1) -> /~{RST}
- U22 pad 11: unconnected-(U22-Pad11) -> /R3-WE
- U23 pad 1: Net-(U23-Pad1) -> /~{R3-OEa}
- U23 pad 19: Net-(U23-Pad1) -> /~{R3-OEa}
- U24 pad 1: Net-(U24-Pad1) -> /~{R3-OEb}
- U24 pad 19: Net-(U24-Pad1) -> /~{R3-OEb}
- U25 pad 1: unconnected-(U25-Pad1) -> /~{RST}
- U25 pad 11: unconnected-(U25-Pad11) -> /ST-WE
- U26 pad 1: Net-(U26-Pad1) -> /~{ST-OEa}
- U26 pad 19: Net-(U26-Pad1) -> /~{ST-OEa}
- U27 pad 1: Net-(U27-Pad1) -> /~{ST-OEb}
- U27 pad 19: Net-(U27-Pad1) -> /~{ST-OEb}
- U28 pad 1: unconnected-(U28-Pad1) -> /~{RST}
- U28 pad 11: unconnected-(U28-Pad11) -> /ST-WE
- U29 pad 1: Net-(U29-Pad1) -> /~{ST-OEa}
- U29 pad 19: Net-(U29-Pad1) -> /~{ST-OEa}
- U3 pad 1: Net-(U2-Pad1) -> /~{R0-OEb}
- U3 pad 19: Net-(U2-Pad1) -> /~{R0-OEb}
- U30 pad 1: Net-(U30-Pad1) -> /~{ST-OEb}
- U30 pad 19: Net-(U30-Pad1) -> /~{ST-OEb}
- U4 pad 1: unconnected-(U4-Pad1) -> /~{RST}
- U4 pad 11: unconnected-(U4-Pad11) -> /R0-WE
- U5 pad 1: Net-(U5-Pad1) -> /~{R0-OEa}
- U5 pad 19: Net-(U5-Pad1) -> /~{R0-OEa}
- U6 pad 1: Net-(U5-Pad1) -> /~{R0-OEb}
- U6 pad 19: Net-(U5-Pad1) -> /~{R0-OEb}
- U7 pad 1: unconnected-(U7-Pad1) -> /~{RST}
- U7 pad 11: unconnected-(U7-Pad11) -> /R1-WE
- U8 pad 1: Net-(U8-Pad1) -> /~{R1-OEa}
- U8 pad 19: Net-(U8-Pad1) -> /~{R1-OEa}
- U9 pad 1: Net-(U8-Pad1) -> /~{R1-OEb}
- U9 pad 19: Net-(U8-Pad1) -> /~{R1-OEb}
Routing:
- net /~{ST-OEb}: track 0.00 -> 32.2 mm
- net /~{R3-OEb}: track 0.00 -> 32.2 mm
- net Net-(U30-Pad1): track 23.5 -> 0.00 mm
- net Net-(U24-Pad1): track 23.5 -> 0.00 mm
- net Net-(U17-Pad1): track 17.4 -> 0.00 mm
- net Net-(U5-Pad1): track 17.4 -> 0.00 mm
- net Net-(U11-Pad1): track 17.4 -> 0.00 mm
- net /~{R1-OEb}: track 0.00 -> 17.4 mm
- net /~{R2-OEb}: track 0.00 -> 17.4 mm
- net /~{R0-OEb}: track 0.00 -> 17.4 mm
- net /~{R2-OEa}: track 0.00 -> 17.3 mm
- net /~{R0-OEa}: track 0.00 -> 17.3 mm
- net Net-(U2-Pad1): track 17.3 -> 0.00 mm
- net Net-(U8-Pad1): track 17.3 -> 0.00 mm
- net Net-(U14-Pad1): track 17.3 -> 0.00 mm
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
Commit message: More development of regfile PCB.
Parts:
- added D104: LED, LED_THT:LED_D5.0mm, F.Cu at (317.5, 373.4)
- added D105: LED, LED_THT:LED_D5.0mm, F.Cu at (311.1, 373.4)
- added D106: LED, LED_THT:LED_D5.0mm, F.Cu at (304.8, 373.4)
- added D107: LED, LED_THT:LED_D5.0mm, F.Cu at (298.4, 373.4)
- added D108: LED, LED_THT:LED_D5.0mm, F.Cu at (292.1, 373.4)
- added D109: LED, LED_THT:LED_D5.0mm, F.Cu at (285.8, 373.4)
- added D110: LED, LED_THT:LED_D5.0mm, F.Cu at (279.4, 373.4)
- added D111: LED, LED_THT:LED_D5.0mm, F.Cu at (273.1, 373.4)
- added D112: LED, LED_THT:LED_D5.0mm, F.Cu at (266.7, 373.4)
- added D113: LED, LED_THT:LED_D5.0mm, F.Cu at (260.4, 373.4)
- added D114: LED, LED_THT:LED_D5.0mm, F.Cu at (254.0, 373.4)
- added D115: LED, LED_THT:LED_D5.0mm, F.Cu at (247.6, 373.4)
- added D116: LED, LED_THT:LED_D5.0mm, F.Cu at (241.3, 373.4)
- added D117: LED, LED_THT:LED_D5.0mm, F.Cu at (234.9, 373.4)
- added D118: LED, LED_THT:LED_D5.0mm, F.Cu at (228.6, 373.4)
- added D119: LED, LED_THT:LED_D5.0mm, F.Cu at (222.2, 373.4)
- added D120: LED, LED_THT:LED_D5.0mm, F.Cu at (317.5, 297.8)
- added D121: LED, LED_THT:LED_D5.0mm, F.Cu at (311.1, 297.8)
- added D122: LED, LED_THT:LED_D5.0mm, F.Cu at (304.8, 297.8)
- added D123: LED, LED_THT:LED_D5.0mm, F.Cu at (298.4, 297.8)
- added D124: LED, LED_THT:LED_D5.0mm, F.Cu at (292.1, 297.8)
- added D125: LED, LED_THT:LED_D5.0mm, F.Cu at (285.7, 297.8)
- added D126: LED, LED_THT:LED_D5.0mm, F.Cu at (279.4, 297.8)
- added D127: LED, LED_THT:LED_D5.0mm, F.Cu at (273.1, 297.8)
- added D128: LED, LED_THT:LED_D5.0mm, F.Cu at (266.7, 297.8)
- added D129: LED, LED_THT:LED_D5.0mm, F.Cu at (260.3, 297.8)
- added D130: LED, LED_THT:LED_D5.0mm, F.Cu at (254.0, 297.8)
- added D131: LED, LED_THT:LED_D5.0mm, F.Cu at (247.6, 297.8)
- added D132: LED, LED_THT:LED_D5.0mm, F.Cu at (241.3, 297.8)
- added D133: LED, LED_THT:LED_D5.0mm, F.Cu at (235.0, 297.8)
- added D134: LED, LED_THT:LED_D5.0mm, F.Cu at (228.6, 297.8)
- added D135: LED, LED_THT:LED_D5.0mm, F.Cu at (222.2, 297.8)
- added R104: R, Resistor_THT:R_Axial_DIN0207_L6.3mm_D2.5mm_P2.54mm_Vertical, F.Cu at (320.0, 379.7)
- added R105: R, Resistor_THT:R_Axial_DIN0207_L6.3mm_D2.5mm_P2.54mm_Vertical, F.Cu at (313.7, 379.7)
- added R106: R, Resistor_THT:R_Axial_DIN0207_L6.3mm_D2.5mm_P2.54mm_Vertical, F.Cu at (307.3, 379.7)
- added R107: R, Resistor_THT:R_Axial_DIN0207_L6.3mm_D2.5mm_P2.54mm_Vertical, F.Cu at (301.0, 379.7)
- added R108: R, Resistor_THT:R_Axial_DIN0207_L6.3mm_D2.5mm_P2.54mm_Vertical, F.Cu at (294.6, 379.7)
- added R109: R, Resistor_THT:R_Axial_DIN0207_L6.3mm_D2.5mm_P2.54mm_Vertical, F.Cu at (288.3, 379.7)
- added R110: R, Resistor_THT:R_Axial_DIN0207_L6.3mm_D2.5mm_P2.54mm_Vertical, F.Cu at (281.9, 379.7)
- added R111: R, Resistor_THT:R_Axial_DIN0207_L6.3mm_D2.5mm_P2.54mm_Vertical, F.Cu at (275.6, 379.7)
- added R112: R, Resistor_THT:R_Axial_DIN0207_L6.3mm_D2.5mm_P2.54mm_Vertical, F.Cu at (269.2, 379.7)
- added R113: R, Resistor_THT:R_Axial_DIN0207_L6.3mm_D2.5mm_P2.54mm_Vertical, F.Cu at (262.9, 379.7)
- added R114: R, Resistor_THT:R_Axial_DIN0207_L6.3mm_D2.5mm_P2.54mm_Vertical, F.Cu at (256.5, 379.7)
- added R115: R, Resistor_THT:R_Axial_DIN0207_L6.3mm_D2.5mm_P2.54mm_Vertical, F.Cu at (250.2, 379.7)
- added R116: R, Resistor_THT:R_Axial_DIN0207_L6.3mm_D2.5mm_P2.54mm_Vertical, F.Cu at (243.8, 379.7)
- added R117: R, Resistor_THT:R_Axial_DIN0207_L6.3mm_D2.5mm_P2.54mm_Vertical, F.Cu at (237.5, 379.7)
- added R118: R, Resistor_THT:R_Axial_DIN0207_L6.3mm_D2.5mm_P2.54mm_Vertical, F.Cu at (231.1, 379.7)
- added R119: R, Resistor_THT:R_Axial_DIN0207_L6.3mm_D2.5mm_P2.54mm_Vertical, F.Cu at (224.8, 379.7)
- added R120: R, Resistor_THT:R_Axial_DIN0207_L6.3mm_D2.5mm_P2.54mm_Vertical, F.Cu at (320.0, 304.2)
- added R121: R, Resistor_THT:R_Axial_DIN0207_L6.3mm_D2.5mm_P2.54mm_Vertical, F.Cu at (313.7, 304.2)
- added R122: R, Resistor_THT:R_Axial_DIN0207_L6.3mm_D2.5mm_P2.54mm_Vertical, F.Cu at (307.3, 304.2)
- added R123: R, Resistor_THT:R_Axial_DIN0207_L6.3mm_D2.5mm_P2.54mm_Vertical, F.Cu at (301.0, 304.2)
- added R124: R, Resistor_THT:R_Axial_DIN0207_L6.3mm_D2.5mm_P2.54mm_Vertical, F.Cu at (294.6, 304.2)
- added R125: R, Resistor_THT:R_Axial_DIN0207_L6.3mm_D2.5mm_P2.54mm_Vertical, F.Cu at (288.3, 304.2)
- added R126: R, Resistor_THT:R_Axial_DIN0207_L6.3mm_D2.5mm_P2.54mm_Vertical, F.Cu at (281.9, 304.2)
- added R127: R, Resistor_THT:R_Axial_DIN0207_L6.3mm_D2.5mm_P2.54mm_Vertical, F.Cu at (275.6, 304.2)
- added R128: R, Resistor_THT:R_Axial_DIN0207_L6.3mm_D2.5mm_P2.54mm_Vertical, F.Cu at (269.2, 304.2)
- added R129: R, Resistor_THT:R_Axial_DIN0207_L6.3mm_D2.5mm_P2.54mm_Vertical, F.Cu at (262.9, 304.2)
- added R130: R, Resistor_THT:R_Axial_DIN0207_L6.3mm_D2.5mm_P2.54mm_Vertical, F.Cu at (256.5, 304.2)
- added R131: R, Resistor_THT:R_Axial_DIN0207_L6.3mm_D2.5mm_P2.54mm_Vertical, F.Cu at (250.2, 304.2)
- added R132: R, Resistor_THT:R_Axial_DIN0207_L6.3mm_D2.5mm_P2.54mm_Vertical, F.Cu at (243.8, 304.2)
- added R133: R, Resistor_THT:R_Axial_DIN0207_L6.3mm_D2.5mm_P2.54mm_Vertical, F.Cu at (237.5, 304.2)
- added R134: R, Resistor_THT:R_Axial_DIN0207_L6.3mm_D2.5mm_P2.54mm_Vertical, F.Cu at (231.1, 304.2)
- added R135: R, Resistor_THT:R_Axial_DIN0207_L6.3mm_D2.5mm_P2.54mm_Vertical, F.Cu at (224.8, 304.2)
- added U52: 74LS00, Package_DIP:DIP-14_W7.62mm, F.Cu at (165.7, 495.9)
- added U53: 74LS273, Package_DIP:DIP-20_W7.62mm, F.Cu at (308.6, 389.3)
- added U54: 74LS273, Package_DIP:DIP-20_W7.62mm, F.Cu at (308.6, 418.5)
- added U55: 74LS273, Package_DIP:DIP-20_W7.62mm, F.Cu at (308.6, 313.7)
- added U56: 74LS273, Package_DIP:DIP-20_W7.62mm, F.Cu at (308.6, 342.9)
- added U57: 74LS244, Package_DIP:DIP-20_W7.62mm, F.Cu at (226.1, 313.7)
- added U58: 74LS244, Package_DIP:DIP-20_W7.62mm, F.Cu at (226.1, 342.9)
- added U59: 74LS244, Package_DIP:DIP-20_W7.62mm, F.Cu at (226.1, 389.3)
- added U60: 74LS244, Package_DIP:DIP-20_W7.62mm, F.Cu at (226.1, 418.5)
- moved U31 649.1 mm to (104.8, 502.9)
- moved U35 634.0 mm to (136.5, 514.3)
- moved U34 628.3 mm to (120.7, 513.7)
- moved J5 584.5 mm to (78.1, 500.4)
- moved J6 583.9 mm to (78.1, 466.1)
- moved U32 582.7 mm to (163.2, 519.1)
- moved U43 531.5 mm to (181.0, 534.7)
- moved R93 506.6 mm to (243.8, 228.6), turned to 180 degrees
- moved U38 504.8 mm to (216.5, 497.2)
- moved U33 504.8 mm to (194.8, 551.2)
- moved U37 504.8 mm to (194.8, 497.2)
- moved U39 504.8 mm to (183.9, 497.2)
- moved U42 504.8 mm to (194.8, 524.2)
- moved U36 504.8 mm to (227.3, 551.2)
- moved U40 504.8 mm to (227.3, 524.2)
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Connections:
- J5 pad 19: unconnected-(J5-Pad19) -> /SImm0
- J5 pad 20: unconnected-(J5-Pad20) -> /SImm1
- U37 pad 10: Net-(U37-Pad10) -> GND
- U38 pad 10: Net-(U37-Pad10) -> GND
- U39 pad 10: Net-(U37-Pad10) -> GND
- U40 pad 10: Net-(U40-Pad10) -> GND
- U41 pad 10: Net-(U40-Pad10) -> GND
- U42 pad 10: Net-(U40-Pad10) -> GND
- U43 pad 10: Net-(U40-Pad10) -> GND
- U48 pad 8: Net-(U48-Pad8) -> GND
- U49 pad 8: Net-(U48-Pad8) -> GND
- U50 pad 10: Net-(U48-Pad8) -> GND
- U51 pad 10: Net-(U48-Pad8) -> GND
Routing:
- net /ImmQb13: track 0.00 -> 153.0 mm
- net /ImmQa13: track 0.00 -> 153.0 mm
- net /ImmQb12: track 0.00 -> 152.4 mm
- net /ImmQa12: track 0.00 -> 152.4 mm
- net /ImmQb15: track 0.00 -> 150.4 mm
- net /ImmQa15: track 0.00 -> 150.4 mm
- net /ImmQb14: track 0.00 -> 149.2 mm
- net /ImmQa14: track 0.00 -> 149.2 mm
- net /ImmQb11: track 0.00 -> 141.4 mm, vias 0 -> 1
- net /ImmQa11: track 0.00 -> 141.4 mm, vias 0 -> 1
- net /ImmQa10: track 0.00 -> 136.3 mm, vias 0 -> 1
- net /ImmQb10: track 0.00 -> 136.3 mm, vias 0 -> 1
- net /ImmQb9: track 0.00 -> 131.2 mm, vias 0 -> 1
- net /ImmQa9: track 0.00 -> 131.2 mm, vias 0 -> 1
- net /ImmQb8: track 0.00 -> 126.1 mm, vias 0 -> 1
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Other:
- board text added: "Imm0"
- board text added: "Imm1"

Commit message: Nearly completed the regfile.
Parts:
- moved J5 579.2 mm to (383.6, 8.27)
- moved J6 493.5 mm to (461.6, 155.6), turned to 180 degrees
- moved U31 440.8 mm to (348.0, 135.2)
- moved U33 421.3 mm to (348.0, 158.8)
- moved U34 421.2 mm to (283.2, 125.1)
- moved U36 410.8 mm to (308.6, 148.6)
- moved U35 384.8 mm to (308.6, 170.2)
- moved D100 369.1 mm to (241.3, 146.7)
- moved D101 369.1 mm to (234.9, 146.7)
- moved D102 369.1 mm to (228.6, 146.7)
- moved D103 369.1 mm to (222.2, 146.7)
- moved D97 369.1 mm to (260.4, 146.7)
- moved D98 369.1 mm to (254.0, 146.7)
- moved D99 369.1 mm to (247.7, 146.7)
- moved R101 369.1 mm to (237.5, 153.0)
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Connections:
- J6 pad 16: GND -> /QZero
- J6 pad 17: GND -> /QUCout
- J6 pad 18: /QZero -> /QSCout
- J6 pad 19: /QUCout -> GND
- J6 pad 20: /QSCout -> GND
- J6 pad 21: /CLK -> GND
- J6 pad 22: /~{RST} -> GND
- U31 pad 9: /~{Imm0-OE} -> /~{Imm-OEa}
- U33 pad 9: /~{Imm1-OE} -> /~{Imm-OEb}
- U40 pad 13: /Db5 -> /Db13
- U40 pad 15: /Db6 -> /Db14
- U40 pad 17: /Db7 -> /Db15
Routing:
- net +5V: track 947.4 -> 2973.6 mm, vias 5 -> 16
- net /~{RST}: track 0.00 -> 1593.8 mm, vias 0 -> 18
- net /~{R0-OEa}: track 62.3 -> 1226.1 mm, vias 1 -> 4
- net /~{R0-OEb}: track 96.7 -> 1238.8 mm, vias 1 -> 4
- net /~{R1-OEa}: track 62.3 -> 1161.7 mm, vias 1 -> 4
- net /~{R1-OEb}: track 96.7 -> 1174.4 mm, vias 1 -> 4
- net /R0-WE: track 0.00 -> 1071.5 mm, vias 0 -> 2
- net /~{R2-OEa}: track 62.3 -> 1097.4 mm, vias 1 -> 4
- net /~{R2-OEb}: track 96.7 -> 1110.1 mm, vias 1 -> 4
- net /R1-WE: track 0.00 -> 996.8 mm, vias 0 -> 3
- net /~{R3-OEa}: track 62.3 -> 1033.0 mm, vias 1 -> 4
- net /~{R3-OEb}: track 96.7 -> 1045.7 mm, vias 1 -> 4
- net /R2-WE: track 0.00 -> 941.2 mm, vias 0 -> 2
- net /~{ST-OEa}: track 62.3 -> 969.4 mm, vias 1 -> 4
- net /~{ST-OEb}: track 96.7 -> 982.1 mm, vias 1 -> 4
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Other:
- board text added: "GND GND GND QSCout QZero GND GND GND GND QIntProg QIRQ GND"
- board text added: "GND GND GND QUCout GND GND GND GND GND QIntSw QNMI GND"
- board text added: "IRQ En."
- board text added: "Int. Prog"
- board text added: "Int. Sw."
- board text added: "NMI En."
- board text added: "PC"
- board text added: "SCout"
- board text added: "UCout"
- board text added: "Zero"

Commit message: Oops! DRC says your design is broken!
Parts:
- moved J5 126.6 mm to (375.3, 134.6), turned to 180 degrees
- moved J6 126.2 mm to (375.3, 63.5)
- moved U33 16.6 mm to (334.0, 167.6)
- moved U31 16.6 mm to (334.0, 144.1)
Connections:
- J5 pad 12: /~{WE} -> /WE
- U32 pad 8: Net-(U32-Pad8) -> /Imm-WEa
- U32 pad 9: /CLK -> Net-(U32-Pad9)
- U35 pad 12: Net-(U32-Pad8) -> Net-(U35-Pad12)
- U35 pad 3: Net-(U32-Pad8) -> Net-(U35-Pad12)
- U35 pad 6: Net-(U32-Pad8) -> Net-(U35-Pad12)
- U36 pad 3: Net-(U32-Pad8) -> Net-(U35-Pad12)
- U36 pad 6: Net-(U32-Pad8) -> Net-(U35-Pad12)
- U36 pad 9: Net-(U32-Pad8) -> Net-(U35-Pad12)
- U52 pad 3: Net-(U52-Pad3) -> Net-(U32-Pad9)
- U52 pad 4: Net-(U52-Pad3) -> /CLK
- U52 pad 5: Net-(U52-Pad3) -> /WE
- U52 pad 6: /Imm-WEa -> Net-(U35-Pad12)
Routing:
- net /B2: track 0.00 -> 229.7 mm, vias 0 -> 3
- net /~{B2}: track 0.00 -> 186.1 mm, vias 0 -> 2
- net /~{A2}: track 0.00 -> 150.0 mm
- net /A2: track 0.00 -> 133.3 mm
- net /B0: track 0.00 -> 91.6 mm, vias 0 -> 1
- net /B1: track 0.00 -> 87.3 mm, vias 0 -> 1
- net Net-(U35-Pad12): track 0.00 -> 78.9 mm, vias 0 -> 4
- net Net-(U32-Pad8): track 70.3 -> 0.00 mm, vias 1 -> 0
- net /~{D2}: track 0.00 -> 66.4 mm
- net /PbA12: track 665.3 -> 722.6 mm
- net /PbA11: track 650.3 -> 703.2 mm
- net /PbA14: track 660.2 -> 712.5 mm
- net /PbA13: track 662.8 -> 714.5 mm
- net /PbA10: track 652.8 -> 701.2 mm
- net /D2: track 0.00 -> 47.2 mm
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
Commit message: Fix most of the tedious DRC errors.
Parts:
- moved D33 1.27 mm to (175.3, 222.2)
- moved D1 1.27 mm to (175.3, 71.1)
- moved D104 1.27 mm to (318.8, 373.4)
- moved D120 1.27 mm to (318.8, 297.8)
- moved D17 1.27 mm to (175.3, 146.7)
- moved D65 1.27 mm to (175.3, 373.4)
- moved D49 1.26 mm to (175.3, 297.8)
- moved D81 1.26 mm to (318.8, 222.2)
- moved D34 1.12 mm to (168.8, 222.2)
- moved D50 1.12 mm to (168.8, 297.8)
- moved D105 1.11 mm to (312.3, 373.4)
- moved D121 1.11 mm to (312.3, 297.8)
- moved D103 1.11 mm to (221.1, 146.7)
- moved D119 1.11 mm to (221.1, 373.4)
- moved D135 1.11 mm to (221.1, 297.8)
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Routing:
- net Net-(D65-Pad2): track 6.35 -> 6.88 mm
- net Net-(D49-Pad2): track 6.35 -> 6.88 mm
- net Net-(D1-Pad2): track 6.35 -> 6.88 mm
- net Net-(D33-Pad2): track 6.35 -> 6.88 mm
- net Net-(D17-Pad2): track 6.35 -> 6.88 mm
- net Net-(D81-Pad2): track 6.35 -> 6.88 mm
- net Net-(D120-Pad2): track 6.35 -> 6.88 mm
- net Net-(D104-Pad2): track 6.35 -> 6.88 mm
