File: kicad/dev/px16_regfile/px16_regfile.kicad_sch (KiCad schematic)
At the start: 201 parts, among them J1 Conn_02x12_Odd_Even, J2 Conn_02x12_Odd_Even, J3 Conn_02x12_Odd_Even, J4 Screw_Terminal_01x02, J5 Conn_02x12_Odd_Even, J6 Conn_02x12_Odd_Even, U1 74LS273, U10 74LS273, U11 74LS244, U12 74LS244, U13 74LS273, U14 74LS244, U15 74LS244, U16 74LS273, U17 74LS244, U18 74LS244, U19 74LS273, U2 74LS244, U20 74LS244, U21 74LS244, U22 74LS273, U23 74LS244, U24 74LS244, U25 74LS273, U26 74LS244, U27 74LS244, U28 74LS273, U29 74LS244, U3 74LS244, U30 74LS244, U31 74LS139, U32 74LS04, U33 74LS139, U34 74LS139, U35 74LS04, U4 74LS273, U5 74LS244, U6 74LS244, U7 74LS273, U8 74LS244, U9 74LS244

Commit message: Work on PC and PF in regfile.
Parts:
- removed U35: 74LS04, symbol 74xx:74LS04
- added D100, D101, D102, D103, D81, D82, D83, D84, D85, D86, D87, D88, D89, D90, D91, D92, D93, D94, D95, D96, D97, D98, D99: LED, LED_THT:LED_D5.0mm, symbol Device:LED
- added R100, R101, R102, R103, R81, R82, R83, R84, R85, R86, R87, R88, R89, R90, R91, R92, R93, R94, R95, R96, R97, R98, R99: R, Resistor_THT:R_Axial_DIN0207_L6.3mm_D2.5mm_P2.54mm_Vertical, symbol Device:R_Small
- added U35, U36: 74LS02, Package_DIP:DIP-14_W7.62mm, symbol 74xx:74LS02
- added U37: 74LS273, Package_DIP:DIP-20_W7.62mm, symbol 74xx:74LS273
- added U38, U39, U40, U41, U42, U43, U46, U47, U50, U51: 74LS244, Package_DIP:DIP-20_W7.62mm, symbol 74xx:74LS244
- added U44, U45, U48, U49: 74LS161, Package_DIP:DIP-16_W7.62mm, symbol 74xx:74LS161
- U31, U33, U34: footprint (none) -> Package_DIP:DIP-16_W7.62mm
- U32: footprint (none) -> Package_DIP:DIP-14_W7.62mm
Connections:
- net +5V: now also U35.14 (VCC), U36.14 (VCC), U37.20 (VCC), U38.20 (VCC), U39.20 (VCC), U40.20 (VCC), U41.20 (VCC), U42.20 (VCC), U43.20 (VCC), U44.16 (VCC), U44.7 (CEP), U45.16 (VCC), U46.20 (VCC), U47.20 (VCC), U48.16 (VCC), U49.16 (VCC), U50.20 (VCC), U51.20 (VCC)
- net CLK: now also U32.9, U44.2 (CP), U45.2 (CP), U48.2 (CP), U49.2 (CP)
- net D2: now also U34.1 (E)
- net Db0: now also U40.2 (I0a), U44.3 (D0)
- net Db1: now also U40.4 (I1a), U44.4 (D1)
- net Db10: now also U48.5 (D2)
- net Db11: now also U48.6 (D3)
- net Db12: now also U49.3 (D0)
- net Db13: now also U49.4 (D1)
- net Db14: now also U49.5 (D2)
- net Db15: now also U49.6 (D3)
- net Db2: now also U40.6 (I2a), U44.5 (D2)
- net Db3: now also U40.8 (I3a), U44.6 (D3)
- net Db4: now also U45.3 (D0)
- net Db5: now also U40.13 (I1b), U45.4 (D1)
- net Db6: now also U40.15 (I2b), U45.5 (D2)
- net Db7: now also U40.17 (I3b), U45.6 (D3)
- net Db8: now also U48.3 (D0)
- net Db9: now also U48.4 (D1)
- net GND: now also D100.1 (K), D101.1 (K), D102.1 (K), D103.1 (K), D81.1 (K), D82.1 (K), D83.1 (K), D84.1 (K), D85.1 (K), D86.1 (K), D87.1 (K), D88.1 (K), D89.1 (K), D90.1 (K), D91.1 (K), D92.1 (K), D93.1 (K), D94.1 (K), D95.1 (K), D96.1 (K), D97.1 (K), D98.1 (K), D99.1 (K), U35.7 (GND), U36.7 (GND), U37.13 (D4), U38.11 (I0b), U38.13 (I1b), U38.15 (I2b), U38.17 (I3b), U39.11 (I0b), U39.13 (I1b), U39.15 (I2b), U39.17 (I3b), U40.11 (I0b), U41.11 (I0b), U42.11 (I0b), U42.2 (I0a), U42.4 (I1a), U42.6 (I2a), U42.8 (I3a), U43.11 (I0b), U43.2 (I0a), U43.4 (I1a), U43.6 (I2a), U43.8 (I3a), U44.8 (GND), U45.8 (GND), U46.10 (GND), U47.10 (GND)
- net IntProg: now also U35.9
- net PF-WE: now also U36.4, U37.11 (Cp)
- net PbA0: now also U38.18 (O0a), U46.18 (O0a)
- net PbA1: now also U38.16 (O1a), U46.16 (O1a)
- net PbA10: now also U42.14 (O2a), U50.14 (O2a)
- net PbA11: now also U42.12 (O3a), U50.12 (O3a)
- net PbA12: now also U42.9 (O0b), U50.9 (O0b)
- net PbA13: now also U42.7 (O1b), U50.7 (O1b)
- net PbA14: now also U42.5 (O2b), U50.5 (O2b)
- net PbA15: now also U42.3 (O3b), U50.3 (O3b)
- net PbA2: now also U38.14 (O2a), U46.14 (O2a)
- net PbA3: now also U38.12 (O3a), U46.12 (O3a)
- net PbA4: now also U38.9 (O0b), U46.9 (O0b)
- net PbA5: now also U38.7 (O1b), U46.7 (O1b)
- net PbA6: now also U38.5 (O2b), U46.5 (O2b)
- net PbA7: now also U38.3 (O3b), U46.3 (O3b)
- net PbA8: now also U42.18 (O0a), U50.18 (O0a)
- net PbA9: now also U42.16 (O1a), U50.16 (O1a)
- net PbB0: now also U39.18 (O0a), U47.18 (O0a)
- net PbB1: now also U39.16 (O1a), U47.16 (O1a)
- net PbB10: now also U43.14 (O2a), U51.14 (O2a)
- net PbB11: now also U43.12 (O3a), U51.12 (O3a)
- net PbB12: now also U43.9 (O0b), U51.9 (O0b)
- net PbB13: now also U43.7 (O1b), U51.7 (O1b)
- net PbB14: now also U43.5 (O2b), U51.5 (O2b)
- net PbB15: now also U43.3 (O3b), U51.3 (O3b)
- net PbB2: now also U39.14 (O2a), U47.14 (O2a)
- net PbB3: now also U39.12 (O3a), U47.12 (O3a)
- net PbB4: now also U39.9 (O0b), U47.9 (O0b)
- net PbB5: now also U39.7 (O1b), U47.7 (O1b)
- net PbB6: now also U39.5 (O2b), U47.5 (O2b)
- net PbB7: now also U39.3 (O3b), U47.3 (O3b)
- net PbB8: now also U43.18 (O0a), U51.18 (O0a)
- net PbB9: now also U43.16 (O1a), U51.16 (O1a)
- net QIRQ: now also R98.2, U37.5 (Q1), U38.4 (I1a), U39.4 (I1a), U41.4 (I1a)
- net QIntProg: now also R100.2, U37.9 (Q3), U38.8 (I3a), U39.8 (I3a), U41.8 (I3a)
- net QIntSw: now also R99.2, U37.6 (Q2), U38.6 (I2a), U39.6 (I2a), U41.6 (I2a)
- net QNMI: now also R97.2, U37.2 (Q0), U38.2 (I0a), U39.2 (I0a), U41.2 (I0a)
- net QSCout: now also R103.2, U37.19 (Q7), U42.17 (I3b), U43.17 (I3b)
- net QUCout: now also R102.2, U37.16 (Q6), U42.15 (I2b), U43.15 (I2b)
- net QZero: now also R101.2, U37.15 (Q5), U42.13 (I1b), U43.13 (I1b)
- net R0-WE: now also U35.1
- net R1-WE: now also U35.4
- net R2-WE: now also U36.10
- net R3-WE: now also U35.13
- net SCout: now also U41.17 (I3b)
- net ST-WE: now also U36.1
- net Zero: now also U41.13 (I1b)
- net ~{D2}: now also U34.15 (E)
- net ~{PC-OEa}: now also U46.1 (OEa), U46.19 (OEb), U50.1 (OEa), U50.19 (OEb)
- net ~{PC-OEb}: now also U47.1 (OEa), U47.19 (OEb), U51.1 (OEa), U51.19 (OEb)
- net ~{PC-WE}: now also U44.9 (~{PE}), U45.9 (~{PE}), U48.9 (~{PE}), U49.9 (~{PE}); no longer U32.9
- net ~{PF-OEa}: now also U38.1 (OEa), U38.19 (OEb), U42.1 (OEa), U42.19 (OEb)
- net ~{PF-OEb}: now also U39.1 (OEa), U39.19 (OEb), U43.1 (OEa), U43.19 (OEb)
- net ~{R0-WE}: now also U35.2
- net ~{R1-WE}: now also U35.5
- net ~{R2-WE}: now also U36.8
- net ~{R3-WE}: now also U35.11
- net ~{RST}: now also U37.1 (~{Mr}), U44.1 (~{MR}), U45.1 (~{MR}), U48.1 (~{MR}), U49.1 (~{MR})
- net ~{ST-WE}: now also U36.2
- net at U32.10: now also U37.14 (D5)
- net at U32.11: now also U35.10
- net PF-Wa: now reaches U32.12
- net PF-Wa: now also U36.11, U41.1 (OEa), U41.19 (OEb)
- net ~{PF-Wa}: now reaches U32.13
- net ~{PF-Wa}: now also U40.1 (OEa), U40.19 (OEb)
- net Inc: now reaches J5.17 (Pin_17)
- net Inc: now also U44.10 (CET), U45.10 (CET), U48.10 (CET), U49.10 (CET)
- net PF-Wb: now reaches J5.18 (Pin_18)
- net PF-Wb: now also U36.12
- net Cout renamed UCout
- net UCout: now also U41.15 (I2b)
- net PC-WE: no longer names the net of U32.8
- net PC-WE: now also U35.12, U35.3, U35.6, U36.3, U36.6, U36.9
- new net: D86.2 (A), R86.1
- new net: U37.10 (GND), U38.10 (GND), U39.10 (GND)
- new net: D99.2 (A), R99.1
- new net: D97.2 (A), R97.1
- new net: D89.2 (A), R89.1
- new net: D88.2 (A), R88.1
- new net: U40.10 (GND), U41.10 (GND), U42.10 (GND), U43.10 (GND)
- new net: D91.2 (A), R91.1
- new net: D100.2 (A), R100.1
- new net: D103.2 (A), R103.1
- new net: U48.15 (TC), U49.7 (CEP)
- new net: U45.15 (TC), U48.7 (CEP)
- new net: U48.8 (GND), U49.8 (GND), U50.10 (GND), U51.10 (GND)
- new net: D93.2 (A), R93.1
- new net: D94.2 (A), R94.1
- new net: D82.2 (A), R82.1
- new net: D95.2 (A), R95.1
- new net: D87.2 (A), R87.1
- new net: D81.2 (A), R81.1
- new net: D96.2 (A), R96.1
- new net: D102.2 (A), R102.1
- new net: D83.2 (A), R83.1
- new net: U44.15 (TC), U45.7 (CEP)
- new net: D101.2 (A), R101.1
- new net: D90.2 (A), R90.1
- new net: U36.13, U36.5
- new net: D92.2 (A), R92.1
- new net: D84.2 (A), R84.1
- new net: D98.2 (A), R98.1
- new net: D85.2 (A), R85.1
- new net DIRQ: U37.4 (D1), U40.16 (O1a), U41.16 (O1a)
- new net DIntProg: U37.8 (D3), U40.12 (O3a), U41.12 (O3a)
- new net DIntSw: U37.7 (D2), U40.14 (O2a), U41.14 (O2a)
- new net DNMI: U37.3 (D0), U40.18 (O0a), U41.18 (O0a)
- new net DSCout: U37.18 (D7), U40.3 (O3b), U41.3 (O3b)
- new net DUCout: U37.17 (D6), U40.5 (O2b), U41.5 (O2b)
- new net DZero: U35.8, U40.7 (O1b), U41.7 (O1b)
- new net PCQ0: R81.2, U44.14 (Q0), U46.2 (I0a), U47.2 (I0a)
- new net PCQ1: R82.2, U44.13 (Q1), U46.4 (I1a), U47.4 (I1a)
- new net PCQ10: R91.2, U48.12 (Q2), U50.6 (I2a), U51.6 (I2a)
- new net PCQ11: R92.2, U48.11 (Q3), U50.8 (I3a), U51.8 (I3a)
- new net PCQ12: R93.2, U49.14 (Q0), U50.11 (I0b), U51.11 (I0b)
- new net PCQ13: R94.2, U49.13 (Q1), U50.13 (I1b), U51.13 (I1b)
- new net PCQ14: R95.2, U49.12 (Q2), U50.15 (I2b), U51.15 (I2b)
- new net PCQ15: R96.2, U49.11 (Q3), U50.17 (I3b), U51.17 (I3b)
- new net PCQ2: R83.2, U44.12 (Q2), U46.6 (I2a), U47.6 (I2a)
- new net PCQ3: R84.2, U44.11 (Q3), U46.8 (I3a), U47.8 (I3a)
- new net PCQ4: R85.2, U45.14 (Q0), U46.11 (I0b), U47.11 (I0b)
- new net PCQ5: R86.2, U45.13 (Q1), U46.13 (I1b), U47.13 (I1b)
- new net PCQ6: R87.2, U45.12 (Q2), U46.15 (I2b), U47.15 (I2b)
- new net PCQ7: R88.2, U45.11 (Q3), U46.17 (I3b), U47.17 (I3b)
- new net PCQ8: R89.2, U48.14 (Q0), U50.2 (I0a), U51.2 (I0a)
- new net PCQ9: R90.2, U48.13 (Q1), U50.4 (I1a), U51.4 (I1a)
Other:
- moved on the sheet: J4, U31C, U32A, U32B, U32C, U32D, U32E, U32F, U32G, U33C, U34C

Commit message: More development of regfile PCB.
Parts:
- added D104, D105, D106, D107, D108, D109, D110, D111, D112, D113, D114, D115, D116, D117, D118, D119, D120, D121, D122, D123, D124, D125, D126, D127, D128, D129, D130, D131, D132, D133, D134, D135: LED, LED_THT:LED_D5.0mm, symbol Device:LED
- added R104, R105, R106, R107, R108, R109, R110, R111, R112, R113, R114, R115, R116, R117, R118, R119, R120, R121, R122, R123, R124, R125, R126, R127, R128, R129, R130, R131, R132, R133, R134, R135: R, Resistor_THT:R_Axial_DIN0207_L6.3mm_D2.5mm_P2.54mm_Vertical, symbol Device:R_Small
- added U52: 74LS00, Package_DIP:DIP-14_W7.62mm, symbol 74xx:74LS00
- added U53, U54, U55, U56: 74LS273, Package_DIP:DIP-20_W7.62mm, symbol 74xx:74LS273
- added U57, U58, U59, U60: 74LS244, Package_DIP:DIP-20_W7.62mm, symbol 74xx:74LS244
Connections:
- net +5V: now also U52.14 (VCC), U53.20 (VCC), U54.20 (VCC), U55.20 (VCC), U56.20 (VCC), U57.20 (VCC), U58.20 (VCC), U59.20 (VCC), U60.20 (VCC)
- net CLK: now also U52.1, U52.9
- net Db0: now also U53.3 (D0), U55.3 (D0)
- net Db1: now also U53.4 (D1), U55.4 (D1)
- net Db10: now also U54.7 (D2), U56.7 (D2)
- net Db11: now also U54.8 (D3), U56.8 (D3)
- net Db12: now also U54.13 (D4), U56.13 (D4)
- net Db13: now also U54.14 (D5), U56.14 (D5)
- net Db14: now also U54.17 (D6), U56.17 (D6)
- net Db15: now also U54.18 (D7), U56.18 (D7)
- net Db2: now also U53.7 (D2), U55.7 (D2)
- net Db3: now also U53.8 (D3), U55.8 (D3)
- net Db4: now also U53.13 (D4), U55.13 (D4)
- net Db5: now also U53.14 (D5), U55.14 (D5)
- net Db6: now also U53.17 (D6), U55.17 (D6)
- net Db7: now also U53.18 (D7), U55.18 (D7)
- net Db8: now also U54.3 (D0), U56.3 (D0)
- net Db9: now also U54.4 (D1), U56.4 (D1)
- net GND: now also U37.10 (GND), U38.10 (GND), U39.10 (GND), U40.10 (GND), U41.10 (GND), U42.10 (GND), U43.10 (GND), U48.8 (GND), U49.8 (GND), U50.10 (GND), U51.10 (GND), D104.1 (K), D105.1 (K), D106.1 (K), D107.1 (K), D108.1 (K), D109.1 (K), D110.1 (K), D111.1 (K), D112.1 (K), D113.1 (K), D114.1 (K), D115.1 (K), D116.1 (K), D117.1 (K), D118.1 (K), D119.1 (K), D120.1 (K), D121.1 (K), D122.1 (K), D123.1 (K), D124.1 (K), D125.1 (K), D126.1 (K), D127.1 (K), D128.1 (K), D129.1 (K), D130.1 (K), D131.1 (K), D132.1 (K), D133.1 (K), D134.1 (K), D135.1 (K), U52.7 (GND), U53.10 (GND), U54.10 (GND), U55.10 (GND), U56.10 (GND), U57.10 (GND), U58.10 (GND), U59.10 (GND), U60.10 (GND)
- net PbA0: now also U57.18 (O0a)
- net PbA1: now also U57.16 (O1a)
- net PbA10: now also U58.14 (O2a)
- net PbA11: now also U58.12 (O3a)
- net PbA12: now also U58.9 (O0b)
- net PbA13: now also U58.7 (O1b)
- net PbA14: now also U58.5 (O2b)
- net PbA15: now also U58.3 (O3b)
- net PbA2: now also U57.14 (O2a)
- net PbA3: now also U57.12 (O3a)
- net PbA4: now also U57.9 (O0b)
- net PbA5: now also U57.7 (O1b)
- net PbA6: now also U57.5 (O2b)
- net PbA7: now also U57.3 (O3b)
- net PbA8: now also U58.18 (O0a)
- net PbA9: now also U58.16 (O1a)
- net PbB0: now also U59.18 (O0a)
- net PbB1: now also U59.16 (O1a)
- net PbB10: now also U60.14 (O2a)
- net PbB11: now also U60.12 (O3a)
- net PbB12: now also U60.9 (O0b)
- net PbB13: now also U60.7 (O1b)
- net PbB14: now also U60.5 (O2b)
- net PbB15: now also U60.3 (O3b)
- net PbB2: now also U59.14 (O2a)
- net PbB3: now also U59.12 (O3a)
- net PbB4: now also U59.9 (O0b)
- net PbB5: now also U59.7 (O1b)
- net PbB6: now also U59.5 (O2b)
- net PbB7: now also U59.3 (O3b)
- net PbB8: now also U60.18 (O0a)
- net PbB9: now also U60.16 (O1a)
- net ~{RST}: now also U53.1 (~{Mr}), U54.1 (~{Mr}), U55.1 (~{Mr}), U56.1 (~{Mr})
- net SImm0: now reaches J5.19 (Pin_19)
- net SImm0: now also U52.2
- net SImm1: now reaches J5.20 (Pin_20)
- net SImm1: now also U52.10
- new net: D113.2 (A), R113.1
- new net: D110.2 (A), R110.1
- new net: D106.2 (A), R106.1
- new net: D130.2 (A), R130.1
- new net: D117.2 (A), R117.1
- new net: D105.2 (A), R105.1
- new net: D122.2 (A), R122.1
- new net: D112.2 (A), R112.1
- new net: D115.2 (A), R115.1
- new net: D123.2 (A), R123.1
- new net: D114.2 (A), R114.1
- new net: D129.2 (A), R129.1
- new net: U52.12, U52.13, U52.8
- new net: D120.2 (A), R120.1
- new net: D128.2 (A), R128.1
- new net: D135.2 (A), R135.1
- new net: D108.2 (A), R108.1
- new net: D126.2 (A), R126.1
- new net: D104.2 (A), R104.1
- new net: D127.2 (A), R127.1
- new net: D109.2 (A), R109.1
- new net: D132.2 (A), R132.1
- new net: U52.3, U52.4, U52.5
- new net: D124.2 (A), R124.1
- new net: D125.2 (A), R125.1
- new net: D134.2 (A), R134.1
- new net: D119.2 (A), R119.1
- new net: D121.2 (A), R121.1
- new net: D116.2 (A), R116.1
- new net: D118.2 (A), R118.1
- new net: D131.2 (A), R131.1
- new net: D133.2 (A), R133.1
- new net: D107.2 (A), R107.1
- new net: D111.2 (A), R111.1
- new net Imm-WEa: U52.6, U53.11 (Cp), U54.11 (Cp)
- new net Imm-WEb: U52.11, U55.11 (Cp), U56.11 (Cp)
- new net ImmQa0: R120.2, U55.2 (Q0), U57.2 (I0a)
- new net ImmQa1: R121.2, U55.5 (Q1), U57.4 (I1a)
- new net ImmQa10: R130.2, U56.6 (Q2), U58.6 (I2a)
- new net ImmQa11: R131.2, U56.9 (Q3), U58.8 (I3a)
- new net ImmQa12: R132.2, U56.12 (Q4), U58.11 (I0b)
- new net ImmQa13: R133.2, U56.15 (Q5), U58.13 (I1b)
- new net ImmQa14: R134.2, U56.16 (Q6), U58.15 (I2b)
- new net ImmQa15: R135.2, U56.19 (Q7), U58.17 (I3b)
- new net ImmQa2: R122.2, U55.6 (Q2), U57.6 (I2a)
- new net ImmQa3: R123.2, U55.9 (Q3), U57.8 (I3a)
- new net ImmQa4: R124.2, U55.12 (Q4), U57.11 (I0b)
- new net ImmQa5: R125.2, U55.15 (Q5), U57.13 (I1b)
- new net ImmQa6: R126.2, U55.16 (Q6), U57.15 (I2b)
- new net ImmQa7: R127.2, U55.19 (Q7), U57.17 (I3b)
- new net ImmQa8: R128.2, U56.2 (Q0), U58.2 (I0a)
- new net ImmQa9: R129.2, U56.5 (Q1), U58.4 (I1a)
- new net ImmQb0: R104.2, U53.2 (Q0), U59.2 (I0a)
- new net ImmQb1: R105.2, U53.5 (Q1), U59.4 (I1a)
- new net ImmQb10: R114.2, U54.6 (Q2), U60.6 (I2a)
- new net ImmQb11: R115.2, U54.9 (Q3), U60.8 (I3a)
- new net ImmQb12: R116.2, U54.12 (Q4), U60.11 (I0b)
- new net ImmQb13: R117.2, U54.15 (Q5), U60.13 (I1b)
- new net ImmQb14: R118.2, U54.16 (Q6), U60.15 (I2b)
- new net ImmQb15: R119.2, U54.19 (Q7), U60.17 (I3b)
- new net ImmQb2: R106.2, U53.6 (Q2), U59.6 (I2a)
- new net ImmQb3: R107.2, U53.9 (Q3), U59.8 (I3a)
- new net ImmQb4: R108.2, U53.12 (Q4), U59.11 (I0b)
- new net ImmQb5: R109.2, U53.15 (Q5), U59.13 (I1b)
- new net ImmQb6: R110.2, U53.16 (Q6), U59.15 (I2b)
- new net ImmQb7: R111.2, U53.19 (Q7), U59.17 (I3b)
- new net ImmQb8: R112.2, U54.2 (Q0), U60.2 (I0a)
- new net ImmQb9: R113.2, U54.5 (Q1), U60.4 (I1a)
- new net ~{Imm-OEa}: U57.1 (OEa), U57.19 (OEb), U58.1 (OEa), U58.19 (OEb)
- new net ~{Imm-OEb}: U59.1 (OEa), U59.19 (OEb), U60.1 (OEa), U60.19 (OEb)
Other:
- title: (none) -> Pixie 16 register file
