File: kicad/dev/px16_regfile_v2/px16_regfile.kicad_pcb (KiCad board)
At the start: 2 copper layers, 229 parts, among them J1 Conn_02x12_Odd_Even, J2 Conn_02x12_Odd_Even, J3 Conn_02x12_Odd_Even, J4 Screw_Terminal_01x02, J5 Conn_02x12_Odd_Even, J6 Conn_02x12_Odd_Even, U1 74LS273, U10 74LS273, U11 74LS244, U12 74LS244, U13 74LS273, U14 74LS244, U15 74LS244, U16 74LS273, U17 74LS244, U18 74LS244, U19 74LS273, U2 74LS244, U20 74LS244, U21 74LS244, U22 74LS273, U23 74LS244, U24 74LS244, U25 74LS273, U26 74LS244, U27 74LS244, U28 74LS273, U29 74LS244, U3 74LS244, U30 74LS244, U31 74LS139, U32 74LS04, U33 74LS139, U34 74LS139, U35 74LS02, U36 74LS02, U37 74LS273, U38 74LS244, U39 74LS244, U4 74LS273, U40 74LS244, U41 74LS244, U42 74LS244, U43 74LS244, U44 74LS161, U45 74LS161, U46 74LS244, U47 74LS244, U48 74LS161, U49 74LS161, U5 74LS244, U50 74LS244, U51 74LS244, U52 74LS00, U53 74LS273, U54 74LS273, U55 74LS273, U56 74LS273, U57 74LS244, U58 74LS244, U59 74LS244, U6 74LS244, U60 74LS244, U7 74LS273, U8 74LS244, U9 74LS244

Commit message: More work on regfile v2
Connections:
- D14 pad 7: /PbA9 -> /ImmQa14
- D14 pad 8: /PbA8 -> /ImmQa15
- D17 pad 5: unconnected-(D17-Pad5) -> /QExFl
- U56 pad 16: /PbA9 -> /ImmQa14
- U56 pad 19: /PbA8 -> /ImmQa15
- U58 pad 15: /PbA9 -> /ImmQa14
- U58 pad 17: /PbA8 -> /ImmQa15
Routing:
- net GND: track 634.1 -> 850.3 mm, vias 23 -> 30
- net +5V: track 658.0 -> 840.5 mm, vias 14 -> 18
- net /~{RST}: track 181.3 -> 285.4 mm, vias 14 -> 20
- net /QExFl: track 31.9 -> 104.5 mm, vias 0 -> 3
- net /CLK: track 0.00 -> 55.3 mm, vias 0 -> 2
- net /QZero: track 32.4 -> 86.6 mm, vias 0 -> 5
- net Net-(U45-Pad15): track 0.00 -> 53.7 mm, vias 0 -> 2
- net /QUCout: track 31.9 -> 83.3 mm, vias 0 -> 3
- net /QSCout: track 32.4 -> 81.8 mm, vias 0 -> 5
- net /LED_GND: track 840.2 -> 884.7 mm, vias 7 -> 8
- net /DNMI: track 0.00 -> 43.5 mm, vias 0 -> 2
- net /~{PF-OEa}: track 0.00 -> 43.4 mm, vias 0 -> 4
- net /DIRQ: track 0.00 -> 43.0 mm, vias 0 -> 2
- net /DIntSw: track 0.00 -> 42.5 mm, vias 0 -> 2
- net /PCQ4: track 54.4 -> 93.7 mm, vias 1 -> 3
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
Commit message: MOAR ((regfile)) ROUTING ((!))
Parts:
- moved U34 270.2 mm to (210.8, 85.7)
- moved U33 239.8 mm to (226.1, 85.7)
- moved U31 212.1 mm to (226.1, 70.5)
- moved U35 197.8 mm to (210.8, 100.3)
- moved U36 197.7 mm to (210.8, 69.8)
- moved U52 148.7 mm to (226.1, 100.3)
- moved J6 68.5 mm to (268.6, 148.0)
- moved J5 40.0 mm to (268.6, 109.9)
Routing:
- net /~{PC-OEb}: track 9.73 -> 169.2 mm, vias 0 -> 4
- net GND: track 850.3 -> 1007.8 mm, vias 30 -> 36
- net /QNMI: track 61.5 -> 154.0 mm, vias 2 -> 5
- net /QIRQ: track 63.4 -> 155.4 mm, vias 4 -> 7
- net /QIntSw: track 62.0 -> 152.0 mm, vias 2 -> 4
- net /Db0: track 117.6 -> 207.4 mm, vias 9 -> 11
- net /Db1: track 120.9 -> 209.3 mm, vias 9 -> 11
- net /QIntProg: track 62.6 -> 149.6 mm, vias 2 -> 4
- net /Db2: track 121.9 -> 207.6 mm, vias 9 -> 11
- net /PF-WE: track 0.00 -> 83.6 mm, vias 0 -> 2
- net /Db3: track 121.2 -> 204.1 mm, vias 9 -> 11
- net /ImmQa15: track 0.00 -> 81.3 mm, vias 0 -> 1
- net /PbA8: track 672.1 -> 590.7 mm, vias 17 -> 16
- net /ImmQa14: track 0.00 -> 81.0 mm, vias 0 -> 1
- net /PbA9: track 647.6 -> 566.6 mm, vias 17 -> 16
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
Commit message: transfer
Routing:
- net /~{PC-WE}: track 31.5 -> 179.0 mm, vias 0 -> 4
- net /~{PC-OEb}: track 169.2 -> 202.3 mm
- net +5V: track 907.1 -> 907.8 mm
