File: kicad/dev/px16_regfile_v2/px16_regfile.kicad_sch (KiCad schematic)
At the start: 228 parts, among them J1 Conn_02x12_Odd_Even, J2 Conn_02x12_Odd_Even, J3 Conn_02x12_Odd_Even, J4 Screw_Terminal_01x02, J5 Conn_02x12_Odd_Even, J6 Conn_02x12_Odd_Even, U1 74LS273, U10 74LS273, U11 74LS244, U12 74LS244, U13 74LS273, U14 74LS244, U15 74LS244, U16 74LS273, U17 74LS244, U18 74LS244, U19 74LS273, U2 74LS244, U20 74LS244, U21 74LS244, U22 74LS273, U23 74LS244, U24 74LS244, U25 74LS273, U26 74LS244, U27 74LS244, U28 74LS273, U29 74LS244, U3 74LS244, U30 74LS244, U31 74LS139, U32 74LS04, U33 74LS139, U34 74LS139, U35 74LS02, U36 74LS02, U37 74LS273, U38 74LS244, U39 74LS244, U4 74LS273, U40 74LS244, U41 74LS244, U42 74LS244, U43 74LS244, U44 74LS161, U45 74LS161, U46 74LS244, U47 74LS244, U48 74LS161, U49 74LS161, U5 74LS244, U50 74LS244, U51 74LS244, U52 74LS00, U53 74LS273, U54 74LS273, U55 74LS273, U56 74LS273, U57 74LS244, U58 74LS244, U59 74LS244, U6 74LS244, U60 74LS244, U7 74LS273, U8 74LS244, U9 74LS244

Commit message: More work on regfile v2
Parts:
- JP1: footprint (none) -> Jumper:SolderJumper-3_P1.3mm_Open_Pad1.0x1.5mm_NumberLabels
Connections:
- net QExFl: now also D17.5 (A)
Changed lines of the file:
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@@
     (stroke (width 0) (type default) (color 0 0 0 0))
   )
+  (wire (pts (xy 518.16 250.19) (xy 527.05 250.19))
+    (stroke (width 0) (type default) (color 0 0 0 0))
+  )
   (wire (pts (xy 274.32 254) (xy 280.67 254))
     (stroke (width 0) (type default) (color 0 0 0 0))
@@
     (effects (font (size 1.27 1.27)) (justify left bottom))
   )
+  (label "QExFl" (at 518.16 250.19 0)
+    (effects (font (size 1.27 1.27)) (justify left bottom))
+  )
   (label "PbA5" (at 228.6 363.22 0)
     (effects (font (size 1.27 1.27)) (justify left bottom))
@@
     (property "Reference" "JP1" (id 0) (at 359.41 166.37 0))
     (property "Value" "SolderJumper_3_Open" (id 1) (at 359.41 168.91 0))
-    (property "Footprint" "" (id 2) (at 359.41 172.72 0)
+    (property "Footprint" "Jumper:SolderJumper-3_P1.3mm_Open_Pad1.0x1.5mm_NumberLabels" (id 2) (at 359.41 172.72 0)
       (effects (font (size 1.27 1.27)) hide)
     )

Commit message: Testing making SPACE for CAPACITOR(s)
Parts:
- added C1: C, symbol Device:C
Connections:
- net Db0: now also C1.1
- net GND: now also C1.2
Changed lines of the file:
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@@
     (stroke (width 0) (type default) (color 0 0 0 0))
   )
+  (wire (pts (xy 49.53 303.53) (xy 54.61 303.53))
+    (stroke (width 0) (type default) (color 0 0 0 0))
+  )
   (wire (pts (xy 495.3 222.25) (xy 501.65 222.25))
     (stroke (width 0) (type default) (color 0 0 0 0))
@@
     (stroke (width 0) (type default) (color 0 0 0 0))
   )
+  (wire (pts (xy 64.77 303.53) (xy 62.23 303.53))
+    (stroke (width 0) (type default) (color 0 0 0 0))
+  )
   (wire (pts (xy 495.3 212.09) (xy 501.65 212.09))
     (stroke (width 0) (type default) (color 0 0 0 0))
@@
     (effects (font (size 1.27 1.27)) (justify left bottom))
   )
+  (label "Db0" (at 49.53 303.53 0)
+    (effects (font (size 1.27 1.27)) (justify left bottom))
+  )
   (label "PbB4" (at 495.3 262.89 0)
     (effects (font (size 1.27 1.27)) (justify left bottom))
@@
     (pin "9")
   )
+  (symbol (lib_id "Device:C") (at 58.42 303.53 90) (unit 1)
+    (in_bom yes) (on_board yes) (fields_autoplaced)
+    (property "Reference" "C1" (id 0) (at 58.42 295.91 90))
+    (property "Value" "C" (id 1) (at 58.42 298.45 90))
+    (property "Footprint" "" (id 2) (at 62.23 302.5648 0)
+      (effects (font (size 1.27 1.27)) hide)
+    )
+    (property "Datasheet" "~" (id 3) (at 58.42 303.53 0)
+      (effects (font (size 1.27 1.27)) hide)
+    )
+    (pin "1")
+    (pin "2")
+  )
   (symbol (lib_id "Device:R_Small") (at 539.75 252.73 90) (unit 1)
     (in_bom yes) (on_board yes)
@@
     (pin "9")
   )
+  (symbol (lib_id "power:GND") (at 64.77 303.53 90) (unit 1)
+    (in_bom yes) (on_board yes) (fields_autoplaced)
+    (property "Reference" "#PWR?" (id 0) (at 71.12 303.53 0)
+      (effects (font (size 1.27 1.27)) hide)
+    )
+    (property "Value" "GND" (id 1) (at 68.58 303.5299 90)
+      (effects (font (size 1.27 1.27)) (justify right))
+    )
+    (property "Footprint" "" (id 2) (at 64.77 303.53 0)
+      (effects (font (size 1.27 1.27)) hide)
+    )
+    (property "Datasheet" "" (id 3) (at 64.77 303.53 0)
+      (effects (font (size 1.27 1.27)) hide)
+    )
+    (pin "1")
+  )
   (symbol (lib_id "power:GND") (at 35.56 30.48 270) (unit 1)
     (in_bom yes) (on_board yes) (fields_autoplaced)
@@
       (reference "#PWR0118") (unit 1) (value "GND") (footprint "")
     )
+    (path "/40719997-575c-46bd-aa98-8050f11fccfb"
+      (reference "#PWR?") (unit 1) (value "GND") (footprint "")
+    )
+    (path "/06d1a66e-0e2e-4e70-8eca-bb252f8bb033"
+      (reference "C1") (unit 1) (value "C") (footprint "Capacitor_SMD:C_0201_0603Metric")
+    )
     (path "/975df1ef-c9c1-4c87-9f58-dc4a36e6c017"

Commit message: The capaciting?
Parts:
- removed C1: C, symbol Device:C
- added C? (x96): C, Capacitor_SMD:C_0201_0603Metric, symbol Device:C
- added J7: Conn_01x02_Male, Connector_PinHeader_2.54mm:PinHeader_1x02_P2.54mm_Vertical, symbol Connector:Conn_01x02_Male
Connections:
- net Db0: now also C?.1, C?.1, C?.1, C?.1, C?.1, C?.1
- net Db1: now also C?.1, C?.1, C?.1, C?.1, C?.1, C?.1
- net Db10: now also C?.1, C?.1, C?.1, C?.1, C?.1, C?.1
- net Db11: now also C?.1, C?.1, C?.1, C?.1, C?.1, C?.1
- net Db12: now also C?.1, C?.1, C?.1, C?.1, C?.1, C?.1
- net Db13: now also C?.1, C?.1, C?.1, C?.1, C?.1, C?.1
- net Db14: now also C?.1, C?.1, C?.1, C?.1, C?.1, C?.1
- net Db15: now also C?.1, C?.1, C?.1, C?.1, C?.1, C?.1
- net Db2: now also C?.1, C?.1, C?.1, C?.1, C?.1, C?.1
- net Db3: now also C?.1, C?.1, C?.1, C?.1, C?.1, C?.1
- net Db4: now also C?.1, C?.1, C?.1, C?.1, C?.1, C?.1
- net Db5: now also C?.1, C?.1, C?.1, C?.1, C?.1, C?.1
- net Db6: now also C?.1, C?.1, C?.1, C?.1, C?.1, C?.1
- net Db7: now also C?.1, C?.1, C?.1, C?.1, C?.1, C?.1
- net Db8: now also C?.1, C?.1, C?.1, C?.1, C?.1, C?.1
- net Db9: now also C?.1, C?.1, C?.1, C?.1, C?.1, C?.1
- net GND: now also C?.2, C?.2, C?.2, C?.2, C?.2, C?.2, C?.2, C?.2, C?.2, C?.2, C?.2, C?.2, C?.2, C?.2, C?.2, C?.2, C?.2, C?.2, C?.2, C?.2, C?.2, C?.2, C?.2, C?.2, C?.2, C?.2, C?.2, C?.2, C?.2, C?.2, C?.2, C?.2, C?.2, C?.2, C?.2, C?.2, C?.2, C?.2, C?.2, C?.2, C?.2, C?.2, C?.2, C?.2, C?.2, C?.2, C?.2, C?.2, C?.2, C?.2, C?.2, C?.2, C?.2, C?.2, C?.2, C?.2, C?.2, C?.2, C?.2, C?.2, C?.2, C?.2, C?.2, C?.2, C?.2, C?.2, C?.2, C?.2, C?.2, C?.2, C?.2, C?.2, C?.2, C?.2, C?.2, C?.2, C?.2, C?.2, C?.2, C?.2, C?.2, C?.2, C?.2, C?.2, C?.2, C?.2, C?.2, C?.2, C?.2, C?.2, C?.2, C?.2, C?.2, C?.2, C?.2, C?.2, J7.1 (Pin_1)
- net LED_GND: now also J7.2 (Pin_2)

Commit message: The capacitanceningification.
Parts:
- added C100, C101, C102, C103, C104, C105, C106, C107, C108, C109, C110, C111, C112, C129, C130, C131, C132, C133, C134, C135, C136, C81, C82, C83, C84, C85, C86, C87, C88, C89, C90, C91, C92, C93, C94, C95, C96, C97, C98, C99: C, Capacitor_SMD:C_0201_0603Metric, symbol Device:C
- gave numbers to parts that had none: 96
Connections:
- net Db0: now also C129.1, C81.1, C97.1
- net Db1: now also C130.1, C82.1, C98.1
- net Db10: now also C107.1, C91.1
- net Db11: now also C108.1, C92.1
- net Db12: now also C109.1, C133.1, C93.1
- net Db13: now also C110.1, C134.1, C94.1
- net Db14: now also C111.1, C135.1, C95.1
- net Db15: now also C112.1, C136.1, C96.1
- net Db2: now also C131.1, C83.1, C99.1
- net Db3: now also C100.1, C132.1, C84.1
- net Db4: now also C101.1, C85.1
- net Db5: now also C102.1, C86.1
- net Db6: now also C103.1, C87.1
- net Db7: now also C104.1, C88.1
- net Db8: now also C105.1, C89.1
- net Db9: now also C106.1, C90.1
- net GND: now also C100.2, C101.2, C102.2, C103.2, C104.2, C105.2, C106.2, C107.2, C108.2, C109.2, C110.2, C111.2, C112.2, C129.2, C130.2, C131.2, C132.2, C133.2, C134.2, C135.2, C136.2, C81.2, C82.2, C83.2, C84.2, C85.2, C86.2, C87.2, C88.2, C89.2, C90.2, C91.2, C92.2, C93.2, C94.2, C95.2, C96.2, C97.2, C98.2, C99.2
Other:
- note added: "Near Imm0"
- note added: "Near Imm1"
- note added: "Near PC"
- note added: "Near PF"
- note added: "Near R0"
- note added: "Near R1"
- note added: "Near R2"
- note added: "Near R3"
- note added: "Near ST"
- moved on the sheet: C1, C10, C11, C113, C114, C115, C116, C117, C118, C119, C12, C120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
